Commit message: modified:   open_manipulator/open_manipulator_description/urdf/open_manipulator_x/open_manipulator_x.urdf modified:   open_manipulator/open_manipulator_description/urdf/open_manipulator_x/open_manipulator_x_arm.urdf.xacro modified:   openmanipulator_task_executor/scripts/open_manipulator_x_pickandplace.py

File: open_manipulator/open_manipulator_description/urdf/open_manipulator_x/open_manipulator_x.urdf (robot description, URDF)
Before this commit: robot open_manipulator_x, 9 links, 8 joints
Joints:
- joint joint3: limit lower=-1.7 upper=1.4 effort=1000 velocity=4.8 -> lower=-1.6 upper=1.4 effort=1000 velocity=4.8

File: open_manipulator/open_manipulator_description/urdf/open_manipulator_x/open_manipulator_x_arm.urdf.xacro (robot description, xacro)
@@ -98,5 +98,5 @@
       <origin xyz="0.024 0 0.128" rpy="0 0 0"/>
       <axis xyz="0 1 0"/>
-      <limit velocity="4.8" effort="1000" lower="${-1.7}" upper="${1.4}" />
+      <limit velocity="4.8" effort="1000" lower="${-1.6}" upper="${1.4}" />
       <dynamics damping="0.1"/>
     </joint>
